File: PCB/Steno.kicad_pcb (KiCad board)
At the start: 4 copper layers, 186.7 x 89.9 mm, 113 parts, among them J1 USB-C USB 2.0 MC-372, Q1 AO3407, SW1 SW_Push_Dual, SW10 H, SW11 R, SW12 O, SW13 *, SW14 E, SW15 #, SW16 F, SW17 R, SW18 U, SW19 P, SW2 #, SW20 B, SW21 *, SW22 #, SW23 L, SW24 G, SW25 T, SW26 S, SW27 D, SW28 Z, SW3 S, SW4 T, SW5 K, SW6 #, SW7 P, SW8 W, SW9 A, U1 BQ27427, U2 BQ24075RGT, U3 MAX16054, U4 TPS709, U5 Conn_01x14_Socket, U6 nRF52840_aQFN73, U7 SSD1306, X1 32.768 kHz, X2 32MHZ

Commit message: try fuel gauge again
Routing:
- net VBUS: track 114.7 -> 114.1 mm
