File: PCB/Steno.kicad_sch (KiCad schematic)
At the start: 111 parts, among them J1 USB-C USB 2.0 MC-372, Q1 AO3407, SW1 SW_Push_Dual, SW10 H, SW11 R, SW12 O, SW13 *, SW14 E, SW15 #, SW16 F, SW17 R, SW18 U, SW19 P, SW2 #, SW20 B, SW21 *, SW22 #, SW23 L, SW24 G, SW25 T, SW26 S, SW27 D, SW28 Z, SW3 S, SW4 T, SW5 K, SW6 #, SW7 P, SW8 W, SW9 A, U1 BQ27427, U2 BQ24075RGT, U3 MAX16054, U4 TPS709, U5 Conn_01x14_Socket, U6 nRF52840_aQFN73, U7 SSD1306, X1 32.768 kHz, X2 32MHZ

Commit message: try fuel gauge again
Parts:
- C30: value 0.1uF -> 100nf
Other:
- note added: "Bluetooth Remove Bond"
- note added: "Bluetooth device 1"
- note added: "Bluetooth device 2"
- note added: "Bluetooth device 3"
- note added: "Bluetooth device 4"
- note added: "Bluetooth device 5"
- note added: "Brightness down"
- note added: "Brightness up"
- note added: "Next song"
- note added: "Pause"
- note added: "Previous song"
- note added: "Vol Up"
- note added: "Vol down"
- note added: "mute"
Changed lines of the file:
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@@
 	(generator_version "9.0")
 	(paper "A4")
+	(text "Previous\nsong"
+		(exclude_from_sim no)
+		(at 469.392 100.33 0)
+		(effects
+			(font
+				(size 1.016 1.016)
+				(color 0 0 0 1)
+			)
+		)
+	)
+	(text "Bluetooth \ndevice 4"
+		(exclude_from_sim no)
+		(at 501.904 89.916 0)
+		(effects
+			(font
+				(size 1.016 1.016)
+				(color 0 0 0 1)
+			)
+		)
+	)
+	(text "Bluetooth \ndevice 2"
+		(exclude_from_sim no)
+		(at 480.314 89.916 0)
+		(effects
+			(font
+				(size 1.016 1.016)
+				(color 0 0 0 1)
+			)
+		)
+	)
+	(text "Next\nsong"
+		(exclude_from_sim no)
+		(at 490.728 100.584 0)
+		(effects
+			(font
+				(size 1.016 1.016)
+				(color 0 0 0 1)
+			)
+		)
+	)
 	(text "USB charge in"
 		(exclude_from_sim no)
@@
 		)
 	)
+	(text "Pause"
+		(exclude_from_sim no)
+		(at 480.06 100.33 0)
+		(effects
+			(font
+				(size 1.016 1.016)
+				(color 0 0 0 1)
+			)
+		)
+	)
+	(text "Bluetooth \ndevice 3"
+		(exclude_from_sim no)
+		(at 490.982 89.916 0)
+		(effects
+			(font
+				(size 1.016 1.016)
+				(color 0 0 0 1)
+			)
+		)
+	)
+	(text "Brightness \ndown"
+		(exclude_from_sim no)
+		(at 437.896 100.584 0)
+		(effects
+			(font
+				(size 1.016 1.016)
+				(color 0 0 0 1)
+			)
+		)
+	)
 	(text "3V REGULATOR"
 		(exclude_from_sim no)
@@
 		)
 	)
+	(text "Bluetooth \ndevice 5"
+		(exclude_from_sim no)
+		(at 512.318 89.916 0)
+		(effects
+			(font
+				(size 1.016 1.016)
+				(color 0 0 0 1)
+			)
+		)
+	)
+	(text "Brightness \nup"
+		(exclude_from_sim no)
+		(at 448.564 100.584 0)
+		(effects
+			(font
+				(size 1.016 1.016)
+				(color 0 0 0 1)
+			)
+		)
+	)
+	(text "Bluetooth \ndevice 1"
+		(exclude_from_sim no)
+		(at 469.646 89.916 0)
+		(effects
+			(font
+				(size 1.016 1.016)
+				(color 0 0 0 1)
+			)
+		)
+	)
 	(text "0x55\n"
 		(exclude_from_sim no)
@@
 		)
 	)
+	(text "mute"
+		(exclude_from_sim no)
+		(at 437.642 90.17 0)
+		(effects
+			(font
+				(size 1.016 1.016)
+				(color 0 0 0 1)
+			)
+		)
+	)
+	(text "Vol Up"
+		(exclude_from_sim no)
+		(at 448.31 89.916 0)
+		(effects
+			(font
+				(size 1.016 1.016)
+				(color 0 0 0 1)
+			)
+		)
+	)
+	(text "Vol down"
+		(exclude_from_sim no)
+		(at 426.72 89.916 0)
+		(effects
+			(font
+				(size 1.016 1.016)
+				(color 0 0 0 1)
+			)
+		)
+	)
+	(text "Bluetooth \nRemove \nBond"
+		(exclude_from_sim no)
+		(at 459.232 94.234 0)
+		(effects
+			(font
+				(size 1.016 1.016)
+				(color 0 0 0 1)
+			)
+		)
+	)
 	(junction
 		(at 207.01 148.59)
@@
 			)
 		)
-		(property "Value" "0.1uF"
+		(property "Value" "100nf"
 			(at 226.06 160.655 0)
 			(effects
